File: Micromouse Power Subsystem.kicad_sch (KiCad schematic)
At the start: 23 parts, among them IC1 CH224K, J1 TYPEC-304-ACP16, J2 Conn_02x16_Odd_Even, J3 B2B-PH-K-S, Q1 NDT3055L, U1 INA219AIDCNR, U2 BQ24074RGTR

Commit message: Added completed schematic for my sections
Parts:
- removed D1: RED/AMBER LED, symbol Device:LED
- removed D2: GREEN LED, symbol Device:LED
- added D1: KT-0805G (GREEN), LED:LED_KT-0603R, symbol KT-0603R:KT-0603R
- added D2: KT-0603R (RED), LED:LED_KT-0603R, symbol KT-0603R:KT-0603R
- C1: value C -> 1µ; footprint (none) -> 1 micro:CAPC3216X180N
- C2, C3: footprint (none) -> 10 micro:CAPC3216X180N
- C4: value C -> 4.7µ; footprint (none) -> 4.7 micro:CAPC2012X140N
- J2: now not fitted
- J3: footprint B2B-PH-K-S:JST_B2B-PH-K-S -> Battery JST Connector:JST_B2B-PH-K-S; now not fitted
- Q1: value NDT3055L -> AO3400A; footprint Package_TO_SOT_SMD:SOT-223-3_TabPin2 -> MOSFET:SOT95P280X125-3N
- R1: footprint Resistor_SMD:R_Shunt_Ohmite_LVK12 -> 100m:RESC6332X65N
- R10: footprint Resistor_SMD:R_Shunt_Ohmite_LVK12 -> 2.2k:RESC1608X55N
- R15: value 190R -> 200R; footprint Resistor_THT:R_Axial_DIN0204_L3.6mm_D1.6mm_P1.90mm_Vertical -> 200 ohm:RESC1608X55N
- R2: footprint Resistor_THT:R_Axial_DIN0204_L3.6mm_D1.6mm_P1.90mm_Vertical -> 6.8k:RESC2012X65N
- R5: footprint Resistor_SMD:R_Shunt_Ohmite_LVK12 -> 4.7k:RESC2012X65N
- R6: footprint Resistor_SMD:R_Shunt_Ohmite_LVK12 -> 10k:RESC2012X65N
- R7: footprint Resistor_SMD:R_Shunt_Ohmite_LVK12 -> 1.2k:RESC2012X65N
- R8, R9: value 100m -> 100R; footprint Resistor_SMD:R_Shunt_Ohmite_LVK12 -> 100 ohm:RESC2012X65N
- U2: footprint BQ24074RGTR:QFN50P300X300X100-17N -> BQ24074:QFN50P300X300X100-17N
Connections:
- net Load is gone; now on net SYS: R1.1, U1.2 (IN-)
- net GND: now also J1.B1-A12 (GND); no longer J1.B4-A9 (GND)
- net SYS: now also D1.A, D2.A
- net at R9.2: now also D1.C
- net at R8.1: now also D2.C
Other:
- note added: "Battery Charging Circuit (Charges at 4.2V)"
